File: prototype/hardware/Kicad/circuit board design.kicad_pcb (KiCad board)
At the start: 4 copper layers, 30.5 x 82.6 mm, 87 parts, among them J1 Conn_01x05, J2 USB_B_Micro, J3 Screw_Terminal_01x04, J4 Conn_01x02, J5 Conn_01x04, J6 Conn_Coaxial, J7 Conn_Coaxial, U1 LSM9DS1, U11 W25Q64JVSSIM, U14 MAX40200AUK, U15 LD3985M33R_TSOT23, U2 0433BM41A0019E, U3 Si4463, U4 MAX-M8Q, U5 H3LIS100DL, U6 Si7232DN, U7 ATSAMD21J18A-AU, U8 MS5607-02BA, U9 STF202-22T1G, X1 TM-32.000-AF3-33-S-Oscillator, Y3 16MHz

Commit message: updated circuit
Parts:
- removed ANT1: Yageo434, flight-computer:Yageo434
- removed BZ1: Buzzer, Buzzer_Beeper:Buzzer_12x9.5RM7.6
- removed C1, C18, C2, C5, C92: 10uF, Capacitor_SMD:C_0603_1608Metric
- removed C10: NF, Capacitor_SMD:C_0402_1005Metric
- removed C11, C15, C16, C17, C23, C25, C3, C4, C6, C7, C89, C91, C93: 100nF, Capacitor_SMD:C_0603_1608Metric
- removed C19, C9: 270pF, Capacitor_SMD:C_0402_1005Metric
- removed C20, C24, C34: 10nF, Capacitor_SMD:C_0603_1608Metric
- removed C21: 33nF, Capacitor_SMD:C_0603_1608Metric
- removed C22, C35, C36, C90: 1uF, Capacitor_SMD:C_0603_1608Metric
- removed C77: 220nF, Capacitor_SMD:C_0603_1608Metric
- removed C8: 10nF, Capacitor_SMD:C_0402_1005Metric
- removed C86, C88: 15pF, Capacitor_SMD:C_0603_1608Metric
- removed D1: RED_LED, LED_SMD:LED_0603_1608Metric
- removed D2: BLUE_LED, LED_SMD:LED_0603_1608Metric
- removed D3: DFLS130L, Diode_SMD:D_PowerDI-123
- removed G***: LOGO, flight-computer:ICSS_Logo
- removed H1, H2, H3, H4: MountingHole_Pad, MountingHole:MountingHole_3.2mm_M3_Pad
- removed J1: Conn_01x05, Connector_PinHeader_2.54mm:PinHeader_1x05_P2.54mm_Vertical
- removed J2: USB_B_Micro, flight-computer:USB_Micro-B_Molex-105017-0001
- removed J3: Screw_Terminal_01x04, flight-computer:TerminalBlock_TE_282834-4_1x04_P2.54mm_Horizontal
- removed J4: Conn_01x02, Connector_JST:JST_PH_B2B-PH-K_1x02_P2.00mm_Vertical
- removed J5: Conn_01x04, flight-computer:NS-Tech_Grove_1x04_P2mm_Vertical
- removed J6, J7: Conn_Coaxial, Connector_Coaxial:U.FL_Hirose_U.FL-R-SMT-1_Vertical
- removed L1: L_Core_Ferrite, Inductor_SMD:L_0603_1608Metric
- removed L2: 27nH, Resistor_SMD:R_0402_1005Metric
- removed L3: 0R, Inductor_SMD:L_0402_1005Metric
- removed L8: 220nH, Inductor_SMD:L_0603_1608Metric
- removed R1, R12, R25, R26: 1.6K, Resistor_SMD:R_0603_1608Metric
- removed R13, R3: 3.3K, Resistor_SMD:R_0603_1608Metric
- removed R15, R28, R29: 120K, Resistor_SMD:R_0603_1608Metric
- removed R16, R6: 27K, Resistor_SMD:R_0603_1608Metric
- removed R2: 10 Ohm, Resistor_SMD:R_0402_1005Metric
- removed R7: NF, Resistor_SMD:R_0402_1005Metric
- removed R8: 4.7K, Resistor_SMD:R_0603_1608Metric
- removed U11: W25Q64JVSSIM, Package_SO:SOIC-8_5.23x5.23mm_P1.27mm
- removed U14: MAX40200AUK, Package_TO_SOT_SMD:SOT-23-5
- removed U15: LD3985M33R_TSOT23, Package_TO_SOT_SMD:TSOT-23-5
- removed U2: 0433BM41A0019E, Johanson_frontend:BALUN_0433BM41A0019E
- removed U4: MAX-M8Q, RF_GPS:ublox_MAX
- removed U5: H3LIS100DL, flight-computer:TFLGA-16_3x3mm
- removed U7: ATSAMD21J18A-AU, Package_QFP:TQFP-64_10x10mm_P0.5mm
- removed U8: MS5607-02BA, Package_LGA:LGA-8_3x5mm_P1.25mm
- removed U9: STF202-22T1G, Package_SO:TSOP-6_1.65x3.05mm_P0.95mm
- removed X1: TM-32.000-AF3-33-S-Oscillator, flight-computer:Crystal_SMD_2520-4Pin_2.5x2.0mm
- removed Y3: 16MHz, flight-computer:Crystal_SMD_2520-4Pin_2.5x2.0mm
- C12: value 10uF -> 100nF
- C14: value 100nF -> 220nF
- R5: value 120K -> 4.7K
- U1: value LSM9DS1 -> MAX-M8C; footprint Package_LGA:LGA-24L_3x3.5mm_P0.43mm -> RF_GPS:ublox_MAX
- U3: value Si4463 -> CMWX1ZZABZ-078; footprint Package_DFN_QFN:QFN-20-1EP_4x4mm_P0.5mm_EP2.6x2.6mm_ThermalVias -> RF_Module:CMWX1ZZABZ
- U6: value Si7232DN -> MS5607-02BA; footprint Package_SO:Vishay_PowerPAK_1212-8_Dual -> Package_LGA:LGA-8_3x5mm_P1.25mm
- moved C13 94.6 mm to (189.4, 122.7), turned to 0 degrees
- moved U1 88.8 mm to (181.0, 127.2), turned to 0 degrees
- moved U6 85.2 mm to (176.9, 136.3), turned to 0 degrees
- moved U3 81.1 mm to (167.6, 128.0), turned to 0 degrees
- moved R5 75.2 mm to (166.6, 138.3), turned to 0 degrees
- moved C14 71.5 mm to (166.6, 135.8), turned to 0 degrees
- moved R4 62.8 mm to (162.5, 138.3), turned to 0 degrees
- moved C12 59.9 mm to (162.5, 135.8), turned to 0 degrees
Connections:
- C13 pad 1: GND -> +3V3
- C13 pad 2: +3V3 -> GND
- C14 pad 1: GND -> +3V3
- C14 pad 2: +3V3 -> GND
- R4 pad 2: /gps/GPS_SDA -> /I2C1_SDA
- R5 pad 1: /MCU/MCU_PA04 -> +3V3
- R5 pad 2: /pyro_driver/FET_A -> /I2C1_SCL
- U1 pad 1: +3V3 -> GND
- U1 pad 10: Net-(U1-Pad10) -> GND
- U1 pad 11: /sensors/ACCL_RDY -> Net-(AE2-Pad1)
- U1 pad 12: /sensors/GYRO_RDY -> GND
- U1 pad 14: GND -> Net-(U1-Pad14)
- U1 pad 15: GND -> Net-(U1-Pad15)
- U1 pad 16: GND -> /I2C1_SDA
- U1 pad 17: GND -> /I2C1_SCL
- U1 pad 18: GND -> /GPS_SAFEBOOT
- U1 pad 2: /gps/GPS_SCL -> Net-(U1-Pad2)
- U1 pad 3: +3V3 -> Net-(U1-Pad3)
- U1 pad 4: /gps/GPS_SDA -> /GPS_TIMEPULSE
- U1 pad 5: +3V3 -> /GPS_EXTINT
- U1 pad 9: /sensors/MAG_RDY -> +3V3
- U3 pad 1: /MCU/MCU_PB11 -> Net-(U3-Pad1)
- U3 pad 10: /MCU/MCU_PA12 -> Net-(U3-Pad10)
- U3 pad 11: /MCU/MCU_PB10 -> Net-(U3-Pad11)
- U3 pad 12: /MCU/MCU_SCLK1 -> Net-(U3-Pad12)
- U3 pad 13: /MCU/MCU_MISO1 -> Net-(U3-Pad13)
- U3 pad 14: /MCU/MCU_MOSI1 -> /GPS_TIMEPULSE
- U3 pad 15: /MCU/MCU_NSEL1 -> /VDD_TCXO
- U3 pad 16: Net-(U3-Pad16) -> /GPS_EXTINT
- U3 pad 17: Net-(C20-Pad1) -> /GPS_SAFEBOOT
- U3 pad 18: GND -> Net-(U3-Pad18)
- U3 pad 21: GND -> Net-(U3-Pad21)
- U3 pad 3: Net-(U2-Pad7) -> GND
- U3 pad 4: Net-(L8-Pad1) -> +3V3
- U3 pad 5: Net-(U3-Pad5) -> +3V3
- U3 pad 7: Net-(U3-Pad7) -> GND
- U3 pad 8: +3V3 -> Net-(U3-Pad8)
- U3 pad 9: /MCU/MCU_PA13 -> Net-(U3-Pad9)
- U6 pad 1: GND -> +3V3
- U6 pad 2: /pyro_driver/FIRE_A -> +3V3
- U6 pad 4: /pyro_driver/FIRE_B -> GND
- U6 pad 5: /pyro_driver/FET_B -> GND
- U6 pad 6: /pyro_driver/FET_A -> Net-(U6-Pad6)
Routing:
- net GND: track 170.7 -> 0.00 mm, vias 53 -> 0
- net +3V3: track 115.3 -> 0.00 mm, vias 25 -> 0
- net /gps/GPS_SCL: track 72.8 -> 0.00 mm, vias 3 -> 0
- net /gps/GPS_SDA: track 60.8 -> 0.00 mm, vias 2 -> 0
- net /MCU/SDA_PA08: track 43.8 -> 0.00 mm, vias 1 -> 0
- net /MCU/SCL_PA09: track 39.7 -> 0.00 mm, vias 1 -> 0
- net /gps/GPS_NRES: track 39.0 -> 0.00 mm, vias 2 -> 0
- net Vdrive: track 38.2 -> 0.00 mm
- net /MCU/MCU_NSEL1: track 36.9 -> 0.00 mm, vias 2 -> 0
- net Net-(C35-Pad1): track 36.7 -> 0.00 mm, vias 2 -> 0
- net /MCU/MCU_PA13: track 34.4 -> 0.00 mm
- net /MCU/MCU_PA12: track 33.6 -> 0.00 mm
- net /gps/GPS_NSAFEBOOT: track 33.6 -> 0.00 mm
- net /MCU/MCU_MISO1: track 32.8 -> 0.00 mm, vias 2 -> 0
- net /pyro_driver/FIRE_A: track 32.6 -> 0.00 mm, vias 2 -> 0
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- removed copper zone on VCC.Cu, net +3V3
- removed copper zone on B.Cu, net GND
- removed copper zone on F.Cu, net GND
- removed copper zone on GND.Cu, net GND
Other:
- board size 30.5 x 82.6 mm -> 35.6 x 26.4 mm
- copper layers 4 -> 2
- board text removed: "Board is 4 layer JLCPCB Type JLC7628 1.6mm overall thickness Layer 1 RF and Signal 1oz copper Insulator .2mm 4.6 dielectric constant Layer 2 Ground 1/2 oz copper Insulator 1.065mm 4.6 dielectric constant Layer 3 Power 1/2oz copper Insulator 0.2mm 4.6 dielectric constant Layer 4 Signal 1oz copper Layer 1-2 50 ohm Microstrip width 11.55mil"
- board text removed: "Rocket Flight Computer v1.1 Imperial College Space Society Medad Newman, Richard Ibbotson 2019"
