File: Tracker_Prototype/hardware/Kicad/circuit board design.sch (KiCad schematic (older format))
At the start: 27 parts, among them J1 Conn_01x06, U1 MAX-M8C, U3 CMWX1ZZABZ-078, U6 MS5607-02BA

Commit message: made some edits to the circuit to remove ERC errors. Added in footprints from Femto
Parts:
- AE1: footprint (none) -> femto_footprints:PAD_3x1.5
- AE2: footprint (none) -> femto_footprints:PAD_3x1.5; symbol Device:Antenna -> flight-computer:GPS_Antenna
- C1, C3, C5: value 0.1uF 0402 -> 100nF; footprint (none) -> Capacitor_SMD:C_0402_1005Metric
- C10, C2: value 10uF 0603 -> 10uF; footprint (none) -> Capacitor_SMD:C_0603_1608Metric
- C11, C9, L1: value NF 0603 -> NF; footprint (none) -> Capacitor_SMD:C_0402_1005Metric
- C12: footprint Capacitor_SMD:C_0603_1608Metric -> Capacitor_SMD:C_0402_1005Metric
- C7: value 1uF 0603 -> 1uF; footprint (none) -> Capacitor_SMD:C_0603_1608Metric
- J1: footprint (none) -> femto_footprints:special_test_pads
- R3: value 10K 0402 -> 10K; footprint (none) -> Resistor_SMD:R_0402_1005Metric
- R4, R5: footprint Resistor_SMD:R_0603_1608Metric -> Resistor_SMD:R_0402_1005Metric
Connections:
- net GND: now also U1.13 (LNA_EN)
- net GPS_TIMEPULSE: now also U3.15 (PB14/SPI2_MISO); no longer U3.14 (PB15/SPI2_MOSI)
- net VDD_TCXO: now also U3.1 (PA12/USB_DP); no longer U3.15 (PB14/SPI2_MISO)
- no-connect marks 30 -> 33
Other:
- note added: "Connect VDD_TCXO to PA12 so that MCU can control \nTCXO on, according to datasheet reference"

Commit message: moved txco power to PB15
Connections:
- net VDD_TCXO: now also U3.14 (PB15/SPI2_MOSI); no longer U3.1 (PA12/USB_DP)
Other:
- note removed: "Connect VDD_TCXO to PA12 so that MCU can control \nTCXO on, according to datasheet reference"
Changed lines of the file:
@@
 Connection ~ 7900 1700
-Wire Wire Line
-	5450 1350 5450 1450
-Connection ~ 5450 1350
-Wire Wire Line
-	5450 1700 4750 1700
-Wire Wire Line
-	5450 1350 4750 1350
-Connection ~ 4750 1350
-Wire Wire Line
-	4750 1350 4750 1450
-$Comp
-L power:+3.3V #PWR?
-U 1 1 5DC840B0
-P 4750 1050
-AR Path="/5D5B15F7/5DC840B0" Ref="#PWR?"  Part="1"
-AR Path="/5DC840B0" Ref="#PWR0109"  Part="1"
-F 0 "#PWR0109" H 4750 900 50  0001 C CNN
-F 1 "+3.3V" H 4765 1223 50  0000 C CNN
-F 2 "" H 4750 1050 50  0001 C CNN
-F 3 "" H 4750 1050 50  0001 C CNN
-	1    4750 1050
-	1    0    0    -1
-$EndComp
-Wire Wire Line
-	4750 1350 4750 1050
-Wire Wire Line
-	5450 1650 5450 1700
-Wire Wire Line
-	4750 1650 4750 1700
-$Comp
-L power:GND #PWR?
-U 1 1 5DC840C5
-P 4750 1850
-AR Path="/5D5B15F7/5DC840C5" Ref="#PWR?"  Part="1"
-AR Path="/5DC840C5" Ref="#PWR0110"  Part="1"
-F 0 "#PWR0110" H 4750 1600 50  0001 C CNN
-F 1 "GND" H 4755 1677 50  0000 C CNN
-F 2 "" H 4750 1850 50  0001 C CNN
-F 3 "" H 4750 1850 50  0001 C CNN
-	1    4750 1850
-	-1   0    0    -1
-$EndComp
-Wire Wire Line
-	4750 1850 4750 1700
-Connection ~ 4750 1700
-Wire Wire Line
-	5450 1350 6050 1350
 Wire Wire Line
 	6450 2250 6900 2250
@@
 Wire Wire Line
 	6150 2250 6150 2400
-Wire Wire Line
-	6050 1350 6050 2400
-Text Label 4900 4000 0    50   ~ 0
-SWDIO
-Text Label 4900 3900 0    50   ~ 0
-VDD_TCXO
-Wire Wire Line
-	5350 3900 4900 3900
 Wire Wire Line
 	13450 6750 13350 6750
@@
 $Comp
 L Device:C_Small C?
-U 1 1 5DC840BE
-P 4750 1550
-AR Path="/5D5B15F7/5DC840BE" Ref="C?"  Part="1"
-AR Path="/5DC840BE" Ref="C2"  Part="1"
-F 0 "C2" H 4842 1596 50  0000 L CNN
-F 1 "10uF" H 4842 1505 50  0000 L CNN
-F 2 "Capacitor_SMD:C_0603_1608Metric" H 4750 1550 50  0001 C CNN
-F 3 "~" H 4750 1550 50  0001 C CNN
-	1    4750 1550
-	-1   0    0    -1
-$EndComp
-$Comp
-L Device:C_Small C?
-U 1 1 5DC840B7
-P 5450 1550
-AR Path="/5D5B15F7/5DC840B7" Ref="C?"  Part="1"
-AR Path="/5DC840B7" Ref="C3"  Part="1"
-F 0 "C3" H 5358 1596 50  0000 R CNN
-F 1 "100nF" H 5358 1505 50  0000 R CNN
-F 2 "Capacitor_SMD:C_0402_1005Metric" H 5450 1550 50  0001 C CNN
-F 3 "~" H 5450 1550 50  0001 C CNN
-	1    5450 1550
-	-1   0    0    -1
-$EndComp
-$Comp
-L Device:C_Small C?
 U 1 1 5DC8409B
 P 7900 1550
@@
 	1    0    0    -1
 $EndComp
-NoConn ~ 7150 3900
 NoConn ~ 5350 5000
 NoConn ~ 6350 2400
@@
 Wire Wire Line
 	5200 8350 5550 8350
-Text Notes 7100 2400 0    50   ~ 0
-Connect VDD_TCXO to PA12 so that MCU can control \nTCXO on, according to datasheet reference
+Text Label 4900 4000 0    50   ~ 0
+SWDIO
+Text Label 7800 3900 2    50   ~ 0
+VDD_TCXO
+Wire Wire Line
+	7150 3900 7800 3900
+NoConn ~ 5350 3900
+Wire Wire Line
+	6050 1350 6050 2400
+$Comp
+L Device:C_Small C?
+U 1 1 5DC840B7
+P 5450 1550
+AR Path="/5D5B15F7/5DC840B7" Ref="C?"  Part="1"
+AR Path="/5DC840B7" Ref="C3"  Part="1"
+F 0 "C3" H 5358 1596 50  0000 R CNN
+F 1 "100nF" H 5358 1505 50  0000 R CNN
+F 2 "Capacitor_SMD:C_0402_1005Metric" H 5450 1550 50  0001 C CNN
+F 3 "~" H 5450 1550 50  0001 C CNN
+	1    5450 1550
+	-1   0    0    -1
+$EndComp
+$Comp
+L Device:C_Small C?
+U 1 1 5DC840BE
+P 4750 1550
+AR Path="/5D5B15F7/5DC840BE" Ref="C?"  Part="1"
+AR Path="/5DC840BE" Ref="C2"  Part="1"
+F 0 "C2" H 4842 1596 50  0000 L CNN
+F 1 "10uF" H 4842 1505 50  0000 L CNN
+F 2 "Capacitor_SMD:C_0603_1608Metric" H 4750 1550 50  0001 C CNN
+F 3 "~" H 4750 1550 50  0001 C CNN
+	1    4750 1550
+	-1   0    0    -1
+$EndComp
+$Comp
+L power:GND #PWR?
+U 1 1 5DC840C5
+P 4750 1850
+AR Path="/5D5B15F7/5DC840C5" Ref="#PWR?"  Part="1"
+AR Path="/5DC840C5" Ref="#PWR0110"  Part="1"
+F 0 "#PWR0110" H 4750 1600 50  0001 C CNN
+F 1 "GND" H 4755 1677 50  0000 C CNN
+F 2 "" H 4750 1850 50  0001 C CNN
+F 3 "" H 4750 1850 50  0001 C CNN
+	1    4750 1850
+	-1   0    0    -1
+$EndComp
+Wire Wire Line
+	5450 1650 5450 1700
+$Comp
+L power:+3.3V #PWR?
+U 1 1 5DC840B0
+P 4750 1050
+AR Path="/5D5B15F7/5DC840B0" Ref="#PWR?"  Part="1"
+AR Path="/5DC840B0" Ref="#PWR0109"  Part="1"
+F 0 "#PWR0109" H 4750 900 50  0001 C CNN
+F 1 "+3.3V" H 4765 1223 50  0000 C CNN
+F 2 "" H 4750 1050 50  0001 C CNN
+F 3 "" H 4750 1050 50  0001 C CNN
+	1    4750 1050
+	1    0    0    -1
+$EndComp
+Wire Wire Line
+	4750 1350 4750 1050
+Wire Wire Line
+	4750 1350 4750 1450
+Connection ~ 4750 1350
+Wire Wire Line
+	4750 1850 4750 1700
+Wire Wire Line
+	4750 1650 4750 1700
+Connection ~ 4750 1700
+Wire Wire Line
+	5450 1700 4750 1700
+Wire Wire Line
+	5450 1350 6050 1350
+Wire Wire Line
+	5450 1350 4750 1350
+Connection ~ 5450 1350
+Wire Wire Line
+	5450 1350 5450 1450
 $EndSCHEMATC

Commit message: changed the footprints for GPS antenna and lora antenna
Parts:
- added J2, J3: Conn_01x01, Connector_PinHeader_1.00mm:PinHeader_1x01_P1.00mm_Vertical, symbol Connector_Generic:Conn_01x01
- AE1, AE2: footprint femto_footprints:PAD_3x1.5 -> Connector_PinHeader_1.00mm:PinHeader_1x01_P1.00mm_Vertical
- SC1, SC2, SC3, SC4, SC5, SC6: footprint (none) -> ~
Connections:
- net +3V3: now also J3.1 (Pin_1)
- net GND: now also J2.1 (Pin_1)
Changed lines of the file:
@@
 $EndComp
-Wire Wire Line
-	1450 9550 1450 8350
 Wire Wire Line
 	1450 8350 2200 8350
@@
 F 0 "SC6" V 4345 8400 50  0000 C CNN
 F 1 "Solar_Cell" V 4436 8400 50  0000 C CNN
-F 2 "" V 4650 8410 50  0001 C CNN
+F 2 "~" V 4650 8410 50  0001 C CNN
 F 3 "~" V 4650 8410 50  0001 C CNN
 	1    4650 8350
@@
 F 0 "SC5" V 3895 8400 50  0000 C CNN
 F 1 "Solar_Cell" V 3986 8400 50  0000 C CNN
-F 2 "" V 4200 8410 50  0001 C CNN
+F 2 "~" V 4200 8410 50  0001 C CNN
 F 3 "~" V 4200 8410 50  0001 C CNN
 	1    4200 8350
@@
 F 0 "SC4" V 3445 8400 50  0000 C CNN
 F 1 "Solar_Cell" V 3536 8400 50  0000 C CNN
-F 2 "" V 3750 8410 50  0001 C CNN
+F 2 "~" V 3750 8410 50  0001 C CNN
 F 3 "~" V 3750 8410 50  0001 C CNN
 	1    3750 8350
@@
 F 0 "SC3" V 2995 8400 50  0000 C CNN
 F 1 "Solar_Cell" V 3086 8400 50  0000 C CNN
-F 2 "" V 3300 8410 50  0001 C CNN
+F 2 "~" V 3300 8410 50  0001 C CNN
 F 3 "~" V 3300 8410 50  0001 C CNN
 	1    3300 8350
@@
 F 0 "SC2" V 2495 8400 50  0000 C CNN
 F 1 "Solar_Cell" V 2586 8400 50  0000 C CNN
-F 2 "" V 2800 8410 50  0001 C CNN
+F 2 "~" V 2800 8410 50  0001 C CNN
 F 3 "~" V 2800 8410 50  0001 C CNN
 	1    2800 8350
@@
 F 0 "SC1" V 1995 8400 50  0000 C CNN
 F 1 "Solar_Cell" V 2086 8400 50  0000 C CNN
-F 2 "" V 2300 8410 50  0001 C CNN
+F 2 "~" V 2300 8410 50  0001 C CNN
 F 3 "~" V 2300 8410 50  0001 C CNN
 	1    2300 8350
@@
 F 0 "AE1" H 8830 4839 50  0000 L CNN
 F 1 "Lora Antenna" H 8830 4748 50  0000 L CNN
-F 2 "femto_footprints:PAD_3x1.5" H 8750 4850 50  0001 C CNN
+F 2 "Connector_PinHeader_1.00mm:PinHeader_1x01_P1.00mm_Vertical" H 8750 4850 50  0001 C CNN
 F 3 "~" H 8750 4850 50  0001 C CNN
 	1    8750 4850
@@
 F 0 "AE2" H 14880 7139 50  0000 L CNN
 F 1 "GPS Antenna" H 14880 7048 50  0000 L CNN
-F 2 "femto_footprints:PAD_3x1.5" H 14800 7150 50  0001 C CNN
+F 2 "Connector_PinHeader_1.00mm:PinHeader_1x01_P1.00mm_Vertical" H 14800 7150 50  0001 C CNN
 F 3 "~" H 14800 7150 50  0001 C CNN
 	1    14800 7150
@@
 Wire Wire Line
 	5450 1350 5450 1450
+Connection ~ 5550 8350
+Wire Wire Line
+	5550 8350 5700 8350
+$Comp
+L Connector_Generic:Conn_01x01 J3
+U 1 1 5DC8A70A
+P 5900 8350
+F 0 "J3" H 5980 8392 50  0000 L CNN
+F 1 "Conn_01x01" H 5980 8301 50  0000 L CNN
+F 2 "Connector_PinHeader_1.00mm:PinHeader_1x01_P1.00mm_Vertical" H 5900 8350 50  0001 C CNN
+F 3 "~" H 5900 8350 50  0001 C CNN
+	1    5900 8350
+	1    0    0    -1
+$EndComp
+$Comp
+L Connector_Generic:Conn_01x01 J2
+U 1 1 5DC8B635
+P 1050 8350
+F 0 "J2" H 968 8125 50  0000 C CNN
+F 1 "Conn_01x01" H 968 8216 50  0000 C CNN
+F 2 "Connector_PinHeader_1.00mm:PinHeader_1x01_P1.00mm_Vertical" H 1050 8350 50  0001 C CNN
+F 3 "~" H 1050 8350 50  0001 C CNN
+	1    1050 8350
+	-1   0    0    1
+$EndComp
+Connection ~ 1450 8350
+Wire Wire Line
+	1450 9550 1450 8350
+Wire Wire Line
+	1250 8350 1450 8350
 $EndSCHEMATC

Commit message: put in solar voltage adc measurments
Parts:
- added J4: 3.3V, Connector_PinHeader_1.00mm:PinHeader_1x01_P1.00mm_Vertical, symbol Connector_Generic:Conn_01x01
- added R1, R2: 100K, Resistor_SMD:R_0402_1005Metric, symbol Device:R
- J2: value Conn_01x01 -> GND
- J3: value Conn_01x01 -> 3.3V
Connections:
- net +3V3: now also R1.1
- net GND: now also R2.2
- net V_SOLAR: now reaches U3.24 (PA2/ADC2)
- net V_SOLAR: now also R1.2, R2.1
- no-connect marks 33 -> 32
Other:
- note added: "Structural plated throughole to hold the guitar wire solar cell structure"
Changed lines of the file:
@@
 Pressure temperature humidity sensor\n
-Wire Notes Line
-	11100 9150 16050 9150
 Wire Notes Line
 	16050 4900 11100 4900
@@
 NoConn ~ 5350 3300
 NoConn ~ 5350 3200
-NoConn ~ 5350 3100
 NoConn ~ 5350 3000
 Wire Wire Line
@@
 Connection ~ 5200 8350
 Wire Wire Line
-	5200 8350 5550 8350
+	5200 8350 5400 8350
 Text Label 4900 4000 0    50   ~ 0
 SWDIO
@@
 P 5900 8350
 F 0 "J3" H 5980 8392 50  0000 L CNN
-F 1 "Conn_01x01" H 5980 8301 50  0000 L CNN
+F 1 "3.3V" H 5980 8301 50  0000 L CNN
 F 2 "Connector_PinHeader_1.00mm:PinHeader_1x01_P1.00mm_Vertical" H 5900 8350 50  0001 C CNN
 F 3 "~" H 5900 8350 50  0001 C CNN
@@
 P 1050 8350
 F 0 "J2" H 968 8125 50  0000 C CNN
-F 1 "Conn_01x01" H 968 8216 50  0000 C CNN
+F 1 "GND" H 968 8216 50  0000 C CNN
 F 2 "Connector_PinHeader_1.00mm:PinHeader_1x01_P1.00mm_Vertical" H 1050 8350 50  0001 C CNN
 F 3 "~" H 1050 8350 50  0001 C CNN
@@
 Wire Wire Line
 	1250 8350 1450 8350
+$Comp
+L Connector_Generic:Conn_01x01 J4
+U 1 1 5DCBAB7A
+P 9150 7650
+F 0 "J4" H 9230 7692 50  0000 L CNN
+F 1 "3.3V" H 9230 7601 50  0000 L CNN
+F 2 "Connector_PinHeader_1.00mm:PinHeader_1x01_P1.00mm_Vertical" H 9150 7650 50  0001 C CNN
+F 3 "~" H 9150 7650 50  0001 C CNN
+	1    9150 7650
+	1    0    0    -1
+$EndComp
+Wire Wire Line
+	5400 8350 5400 8700
+Connection ~ 5400 8350
+Wire Wire Line
+	5400 8350 5550 8350
+$Comp
+L power:GND #PWR01
+U 1 1 5DCCDF86
+P 5400 9600
+F 0 "#PWR01" H 5400 9350 50  0001 C CNN
+F 1 "GND" H 5405 9427 50  0000 C CNN
+F 2 "" H 5400 9600 50  0001 C CNN
+F 3 "" H 5400 9600 50  0001 C CNN
+	1    5400 9600
+	1    0    0    -1
+$EndComp
+$Comp
+L Device:R R1
+U 1 1 5DCCF4D3
+P 5400 8850
+F 0 "R1" H 5470 8896 50  0000 L CNN
+F 1 "100K" H 5470 8805 50  0000 L CNN
+F 2 "Resistor_SMD:R_0402_1005Metric" V 5330 8850 50  0001 C CNN
+F 3 "~" H 5400 8850 50  0001 C CNN
+	1    5400 8850
+	1    0    0    -1
+$EndComp
+Wire Wire Line
+	5400 9000 5400 9100
+$Comp
+L Device:R R2
+U 1 1 5DCD0192
+P 5400 9350
+F 0 "R2" H 5470 9396 50  0000 L CNN
+F 1 "100K" H 5470 9305 50  0000 L CNN
+F 2 "Resistor_SMD:R_0402_1005Metric" V 5330 9350 50  0001 C CNN
+F 3 "~" H 5400 9350 50  0001 C CNN
+	1    5400 9350
+	1    0    0    -1
+$EndComp
+Wire Wire Line
+	5400 9500 5400 9600
+Wire Wire Line
+	5400 9100 6050 9100
+Connection ~ 5400 9100
+Wire Wire Line
+	5400 9100 5400 9200
+Text Label 6050 9100 2    50   ~ 0
+V_SOLAR
+Wire Notes Line
+	6950 9150 16050 9150
+Text Notes 7650 8400 0    50   ~ 0
+Structural plated throughole to hold the guitar wire solar cell structure
+Wire Wire Line
+	5350 3100 4900 3100
+Text Label 4900 3100 0    50   ~ 0
+V_SOLAR
 $EndSCHEMATC

Commit message: Fully routed the board
Parts:
- removed C2: 10uF, Capacitor_SMD:C_0603_1608Metric, symbol Device:C_Small
- removed C3: 100nF, Capacitor_SMD:C_0402_1005Metric, symbol Device:C_Small
- AE1, AE2, J2, J3: footprint Connector_PinHeader_1.00mm:PinHeader_1x01_P1.00mm_Vertical -> Connector_Wire:SolderWirePad_1x01_Drill0.8mm
- J4: value 3.3V -> Unconnected; footprint Connector_PinHeader_1.00mm:PinHeader_1x01_P1.00mm_Vertical -> Connector_Wire:SolderWirePad_1x01_Drill0.8mm
Connections:
- net VDD_TCXO: now also U3.1 (PA12/USB_DP); no longer U3.14 (PB15/SPI2_MOSI)
- no-connect marks 32 -> 34
Changed lines of the file:
@@
 NoConn ~ 7150 4900
 NoConn ~ 7150 5000
-NoConn ~ 5350 3700
 NoConn ~ 5350 3600
 NoConn ~ 5350 3500
@@
 F 0 "AE1" H 8830 4839 50  0000 L CNN
 F 1 "Lora Antenna" H 8830 4748 50  0000 L CNN
-F 2 "Connector_PinHeader_1.00mm:PinHeader_1x01_P1.00mm_Vertical" H 8750 4850 50  0001 C CNN
+F 2 "Connector_Wire:SolderWirePad_1x01_Drill0.8mm" H 8750 4850 50  0001 C CNN
 F 3 "~" H 8750 4850 50  0001 C CNN
 	1    8750 4850
@@
 F 0 "AE2" H 14880 7139 50  0000 L CNN
 F 1 "GPS Antenna" H 14880 7048 50  0000 L CNN
-F 2 "Connector_PinHeader_1.00mm:PinHeader_1x01_P1.00mm_Vertical" H 14800 7150 50  0001 C CNN
+F 2 "Connector_Wire:SolderWirePad_1x01_Drill0.8mm" H 14800 7150 50  0001 C CNN
 F 3 "~" H 14800 7150 50  0001 C CNN
 	1    14800 7150
@@
 Text Label 4900 4000 0    50   ~ 0
 SWDIO
-Text Label 7800 3900 2    50   ~ 0
+Text Label 4900 3900 0    50   ~ 0
 VDD_TCXO
 Wire Wire Line
-	7150 3900 7800 3900
-NoConn ~ 5350 3900
+	5350 3900 4900 3900
 Wire Wire Line
 	6050 1350 6050 2400
-$Comp
-L Device:C_Small C?
-U 1 1 5DC840B7
-P 5450 1550
-AR Path="/5D5B15F7/5DC840B7" Ref="C?"  Part="1"
-AR Path="/5DC840B7" Ref="C3"  Part="1"
-F 0 "C3" H 5358 1596 50  0000 R CNN
-F 1 "100nF" H 5358 1505 50  0000 R CNN
-F 2 "Capacitor_SMD:C_0402_1005Metric" H 5450 1550 50  0001 C CNN
-F 3 "~" H 5450 1550 50  0001 C CNN
-	1    5450 1550
-	-1   0    0    -1
-$EndComp
-$Comp
-L Device:C_Small C?
-U 1 1 5DC840BE
-P 4750 1550
-AR Path="/5D5B15F7/5DC840BE" Ref="C?"  Part="1"
-AR Path="/5DC840BE" Ref="C2"  Part="1"
-F 0 "C2" H 4842 1596 50  0000 L CNN
-F 1 "10uF" H 4842 1505 50  0000 L CNN
-F 2 "Capacitor_SMD:C_0603_1608Metric" H 4750 1550 50  0001 C CNN
-F 3 "~" H 4750 1550 50  0001 C CNN
-	1    4750 1550
-	-1   0    0    -1
-$EndComp
-$Comp
-L power:GND #PWR?
-U 1 1 5DC840C5
-P 4750 1850
-AR Path="/5D5B15F7/5DC840C5" Ref="#PWR?"  Part="1"
-AR Path="/5DC840C5" Ref="#PWR0110"  Part="1"
-F 0 "#PWR0110" H 4750 1600 50  0001 C CNN
-F 1 "GND" H 4755 1677 50  0000 C CNN
-F 2 "" H 4750 1850 50  0001 C CNN
-F 3 "" H 4750 1850 50  0001 C CNN
-	1    4750 1850
-	-1   0    0    -1
-$EndComp
-Wire Wire Line
-	5450 1650 5450 1700
 $Comp
 L power:+3.3V #PWR?
@@
 Wire Wire Line
 	4750 1350 4750 1050
-Wire Wire Line
-	4750 1350 4750 1450
-Connection ~ 4750 1350
-Wire Wire Line
-	4750 1850 4750 1700
-Wire Wire Line
-	4750 1650 4750 1700
-Connection ~ 4750 1700
-Wire Wire Line
-	5450 1700 4750 1700
-Wire Wire Line
-	5450 1350 6050 1350
-Wire Wire Line
-	5450 1350 4750 1350
-Connection ~ 5450 1350
-Wire Wire Line
-	5450 1350 5450 1450
 Connection ~ 5550 8350
 Wire Wire Line
@@
 F 0 "J3" H 5980 8392 50  0000 L CNN
 F 1 "3.3V" H 5980 8301 50  0000 L CNN
-F 2 "Connector_PinHeader_1.00mm:PinHeader_1x01_P1.00mm_Vertical" H 5900 8350 50  0001 C CNN
+F 2 "Connector_Wire:SolderWirePad_1x01_Drill0.8mm" H 5900 8350 50  0001 C CNN
 F 3 "~" H 5900 8350 50  0001 C CNN
 	1    5900 8350
@@
 F 0 "J2" H 968 8125 50  0000 C CNN
 F 1 "GND" H 968 8216 50  0000 C CNN
-F 2 "Connector_PinHeader_1.00mm:PinHeader_1x01_P1.00mm_Vertical" H 1050 8350 50  0001 C CNN
+F 2 "Connector_Wire:SolderWirePad_1x01_Drill0.8mm" H 1050 8350 50  0001 C CNN
 F 3 "~" H 1050 8350 50  0001 C CNN
 	1    1050 8350
@@
 P 9150 7650
 F 0 "J4" H 9230 7692 50  0000 L CNN
-F 1 "3.3V" H 9230 7601 50  0000 L CNN
-F 2 "Connector_PinHeader_1.00mm:PinHeader_1x01_P1.00mm_Vertical" H 9150 7650 50  0001 C CNN
+F 1 "Unconnected" H 9230 7601 50  0000 L CNN
+F 2 "Connector_Wire:SolderWirePad_1x01_Drill0.8mm" H 9150 7650 50  0001 C CNN
 F 3 "~" H 9150 7650 50  0001 C CNN
 	1    9150 7650
@@
 Text Label 4900 3100 0    50   ~ 0
 V_SOLAR
+Wire Wire Line
+	4750 1350 6050 1350
+NoConn ~ 7150 3900
+NoConn ~ 5350 3700
+NoConn ~ 8950 7650
+NoConn ~ 9800 3250
 $EndSCHEMATC

Commit message: Changed the TCXO power pin. Changed the track width for RF transmission lines to 0.86mm
Connections:
- net VDD_TCXO: now also U3.14 (PB15/SPI2_MOSI); no longer U3.1 (PA12/USB_DP)
- no-connect marks 34 -> 33
Changed lines of the file:
@@
 Text Label 4900 4000 0    50   ~ 0
 SWDIO
-Text Label 4900 3900 0    50   ~ 0
+Text Label 7800 3900 2    50   ~ 0
 VDD_TCXO
 Wire Wire Line
-	5350 3900 4900 3900
+	7150 3900 7800 3900
 Wire Wire Line
 	6050 1350 6050 2400
@@
 Wire Wire Line
 	4750 1350 6050 1350
-NoConn ~ 7150 3900
 NoConn ~ 5350 3700
 NoConn ~ 8950 7650
-NoConn ~ 9800 3250
+NoConn ~ 5350 3900
 $EndSCHEMATC
