File: Tracker_Prototype/hardware/Kicad/Picotracker V1a/_autosave-circuit board design.kicad_pcb (KiCad board)
At the start: 2 copper layers, 33.3 x 20.1 mm, 29 parts, among them J1 Conn_01x06, J2 GND, J3 3.3V, SW1 SW_Push, U1 MAX-M8C, U3 CMWX1ZZABZ-078, U6 MS5607-02BA

Commit message: finished the layout of the simple version a
Parts:
- added G***: LOGO, flight-computer:ICSS_Logo, B.Cu at (281.8, 170.4)
Routing:
- net GND: track 86.3 -> 79.3 mm, vias 9 -> 8
- net Net-(C9-Pad1): track 8.96 -> 11.0 mm
- net /GPS_SAFEBOOT: track 8.16 -> 9.36 mm
