File: Tracker_Prototype/hardware/Kicad/Picotracker V1b/circuit board design.sch (KiCad schematic (older format))
At the start: 35 parts, among them J1 Conn_01x06, J2 GND, J3 3.3V, SW1 SW_Push, U1 MAX-M8C, U3 CMWX1ZZABZ-078, U6 MS5607-02BA

Commit message: added in the libraries to the b variant from femto
Parts:
- removed AE2: GPS Antenna, Connector_Wire:SolderWirePad_1x01_Drill0.8mm, symbol flight-computer:GPS_Antenna
- removed C12: 100nF, Capacitor_SMD:C_0402_1005Metric, symbol Device:C_Small
- removed C13: 10uF, Capacitor_SMD:C_0603_1608Metric, symbol Device:C_Small
- removed U1: MAX-M8C, RF_GPS:ublox_MAX, symbol RF_GPS:MAX-M8C
- added IC1: ZOE-M8G, flight-computer:ZOE-M8, symbol femto-lib:ZOE-M8G
Connections:
- wire segments 132 -> 105
- no-connect marks 31 -> 28
Other:
- note added: "Structural plated throughole to \nhold the guitar wire solar \ncell structure"
- note removed: "Structural plated throughole to hold the guitar wire solar cell structure"
- moved on the sheet: SolarCellMount1, StringHole1

Commit message: updated the "b" variant
Parts:
- removed IC1: ZOE-M8G, flight-computer:ZOE-M8, symbol femto-lib:ZOE-M8G
- removed R1, R2: 100K, Resistor_SMD:R_0402_1005Metric, symbol Device:R
- removed SC1, SC2, SC3, SC4, SC5, SC6: Solar_Cell, ~, symbol Device:Solar_Cell
- added C16: 1n, pecanpico:C_0402, symbol pecanpico:C
- added C17, C3: 22u, pecanpico:C_0805, symbol pecanpico:C
- added C18: 100n, pecanpico:C_0402, symbol pecanpico:C
- added D2: LED, pecanpico:LED_0402, symbol Device:LED
- added IC7: SPV1040, Package_SO:TSSOP-8_4.4x3mm_P0.65mm, symbol pecanpico:SPV1040
- added IC8: SIP32431DNP3-T1GE4, pecanpico:DFN-4-1EP_1.2x1.6mm_P0.5mm_EP, symbol pecanpico:SIP3243x
- added IC9: ZOE-M8G/B, pecanpico:ZOE-M8, symbol pecanpico:ZOE-M8G
- added J4: Conn_01x01, Connector_PinHeader_1.27mm:PinHeader_1x01_P1.27mm_Vertical, symbol Connector_Generic:Conn_01x01
- added L7: XFL2006-472MEB, pecanpico:XFL20xx, symbol pecanpico:L_Small
- added R1, R8: R, pecanpico:R_0402, symbol pecanpico:R
- J3: value 3.3V -> +SOL
Connections:
- net labels added: +1V8, +GPS, +SOL, GPS_EN, MISO, MOSI, SCK2, ~CS_GPS
- wire segments 105 -> 187
Other:
- note removed: "0.5V solar cells"
- moved on the sheet: J3

Commit message: mostly wired up the "b" variant. Changed the fill clearance for copper pour for the "a" variant to a much smaller 0.15mm
Parts:
- removed D2: LED, pecanpico:LED_0402, symbol Device:LED
- added BT?: Battery_Cell, symbol Device:Battery_Cell
- added R2, R9: 10K, Resistor_SMD:R_0402_1005Metric, symbol Device:R
- C16, C18: footprint pecanpico:C_0402 -> Capacitor_SMD:C_0402_1005Metric
- C17, C3: footprint pecanpico:C_0805 -> Capacitor_SMD:C_0805_2012Metric
- R1, R8: footprint pecanpico:R_0402 -> Resistor_SMD:R_0402_1005Metric
Connections:
- net +1V8 is gone; now on net +3V3: IC8.3 (IN)
- net SCK2 is gone; now on net I2C1_SCL: IC9.B1 (SCL/SPI_CLK)
- net ~CS_GPS is gone; now on net I2C1_SDA: IC9.A2 (SDA/SPI_~CS)
- net +3V3: now also BT?.1 (+)
- net +SOL: now also R2.1
- net GND: now also BT?.2 (-), R9.2
- net GPS_EN: now also U3.38 (PB7/LPTIM1_IN2)
- net GPS_EXTINT: now also IC9.G4 (PIO13/EXTINT)
- net GPS_SAFEBOOT: now also IC9.C4 (~SAFEBOOT)
- net V_SOLAR: now also R2.2, R9.1
- net GPS_TIMEPULSE: no longer names the net of U3.15 (PB14/SPI2_MISO)
- net MISO: no longer names the net of IC9.J5 (TXD/SPI_MISO)
- net MOSI: no longer names the net of IC9.J4 (RXD/SPI_MOSI)
- no-connect marks 28 -> 46
Other:
- note added: "MPPT + boost converter to charge battery"
- note added: "Solar Connection\n\n"
- note added: "Switch to turn on and off GPS\n"
- note removed: "Ok, it is not as simple as this. -Medad 21/10/19"
- note removed: "Power supply\n"
Changed lines of the file:
@@
 GPS circuit\n
-Wire Notes Line
-	500  11200 6950 11200
 Wire Notes Line
 	500  6850 500  11200
 Text Notes 650  11100 0    50   ~ 0
-Power supply\n
+Solar Connection\n\n
 Text Label 7800 3400 2    50   ~ 0
 I2C1_SCL
@@
 Text Label 12000 2200 0    50   ~ 0
 I2C1_SCL
-$Comp
-L power:GND #PWR0102
-U 1 1 5DEE121A
-P 1450 8750
-F 0 "#PWR0102" H 1450 8500 50  0001 C CNN
-F 1 "GND" H 1455 8577 50  0000 C CNN
-F 2 "" H 1450 8750 50  0001 C CNN
-F 3 "" H 1450 8750 50  0001 C CNN
-	1    1450 8750
-	1    0    0    -1
-$EndComp
-Text Notes 3050 10200 0    50   ~ 0
-Ok, it is not as simple as this. -Medad 21/10/19
 Wire Wire Line
 	6450 2400 6450 2250
@@
 GPS_EXTINT
 NoConn ~ 7150 3000
-NoConn ~ 7150 3300
 NoConn ~ 7150 4100
 NoConn ~ 7150 4200
@@
 NoConn ~ 5350 3200
 NoConn ~ 5350 3000
-Wire Wire Line
-	7150 3800 7800 3800
-Text Label 7800 3800 2    50   ~ 0
-GPS_TIMEPULSE
 NoConn ~ 5350 4800
 NoConn ~ 5350 4700
@@
 Wire Notes Line
 	550  650  16050 650
-Wire Notes Line
-	11100 650  11100 9150
 Wire Notes Line
 	16050 650  16050 9150
@@
 	-1   0    0    1
 $EndComp
-Wire Wire Line
-	1450 8750 1450 8350
-Wire Wire Line
-	1250 8350 1450 8350
 $Comp
 L Connector_Generic:Conn_01x01 SolarCellMount1
@@
 Connection ~ 6250 2250
 Wire Wire Line
-	1250 7950 1450 7950
-Wire Wire Line
-	1450 7950 1450 7450
+	1250 7950 1300 7950
 $Comp
 L femto-lib:+SOL #PWR0134
 U 1 1 5DCC7320
-P 1450 7450
-F 0 "#PWR0134" H 1450 7300 50  0001 C CNN
-F 1 "+SOL" H 1465 7623 50  0000 C CNN
-F 2 "" H 1450 7450 50  0000 C CNN
-F 3 "" H 1450 7450 50  0000 C CNN
-	1    1450 7450
+P 2400 7450
+F 0 "#PWR0134" H 2400 7300 50  0001 C CNN
+F 1 "+SOL" H 2415 7623 50  0000 C CNN
+F 2 "" H 2400 7450 50  0000 C CNN
+F 3 "" H 2400 7450 50  0000 C CNN
+	1    2400 7450
 	1    0    0    -1
 $EndComp
@@
 F 0 "C3" V 8050 8150 50  0000 R CNN
 F 1 "22u" V 8050 8250 50  0000 L CNN
-F 2 "pecanpico:C_0805" H 8138 8050 50  0001 C CNN
+F 2 "Capacitor_SMD:C_0805_2012Metric" H 8138 8050 50  0001 C CNN
 F 3 "" H 8100 8200 50  0001 C CNN
 	1    8100 8200
@@
 F 0 "R8" V 9600 8200 50  0000 C CNN
 F 1 "R" V 9700 8200 50  0000 C CNN
-F 2 "pecanpico:R_0402" V 9630 8200 50  0001 C CNN
+F 2 "Resistor_SMD:R_0402_1005Metric" V 9630 8200 50  0001 C CNN
 F 3 "" H 9700 8200 50  0001 C CNN
 	1    9700 8200
@@
 F 0 "R1" V 9600 7900 50  0000 C CNN
 F 1 "R" V 9700 7900 50  0000 C CNN
-F 2 "pecanpico:R_0402" V 9630 7900 50  0001 C CNN
+F 2 "Resistor_SMD:R_0402_1005Metric" V 9630 7900 50  0001 C CNN
 F 3 "" H 9700 7900 50  0001 C CNN
 	1    9700 7900
@@
 F 0 "C17" V 9950 8000 50  0000 R CNN
 F 1 "22u" V 9950 8100 50  0000 L CNN
-F 2 "pecanpico:C_0805" H 10038 7900 50  0001 C CNN
+F 2 "Capacitor_SMD:C_0805_2012Metric" H 10038 7900 50  0001 C CNN
 F 3 "" H 10000 8050 50  0001 C CNN
 	1    10000 8050
@@
 F 0 "C16" V 9450 8200 50  0000 R CNN
 F 1 "1n" V 9450 8300 50  0000 L CNN
-F 2 "pecanpico:C_0402" H 9538 8100 50  0001 C CNN
+F 2 "Capacitor_SMD:C_0402_1005Metric" H 9538 8100 50  0001 C CNN
 F 3 "" H 9500 8250 50  0001 C CNN
 	1    9500 8250
@@
 Wire Wire Line
 	14550 5600 14350 5600
-Wire Wire Line
-	14350 6700 14750 6700
-Wire Wire Line
-	14750 6800 14350 6800
 $Comp
 L pecanpico:C C?
@@
 F 0 "C18" V 12700 6200 50  0000 R CNN
 F 1 "100n" V 12700 6300 50  0000 L CNN
-F 2 "pecanpico:C_0402" H 12788 6100 50  0001 C CNN
+F 2 "Capacitor_SMD:C_0402_1005Metric" H 12788 6100 50  0001 C CNN
 F 3 "" H 12750 6250 50  0001 C CNN
 	1    12750 6250
@@
 	14450 7200 14450 7600
 Connection ~ 14450 7600
-Wire Wire Line
-	14350 6600 14750 6600
-Wire Wire Line
-	14350 6500 14750 6500
-Text Label 14750 6700 2    50   ~ 0
-MOSI
-Text Label 14750 6800 2    50   ~ 0
-MISO
-Text Label 14750 6500 2    50   ~ 0
-~CS_GPS
-$Comp
-L Device:LED D?
-U 1 1 5DDC92C2
-P 14700 7300
-AR Path="/5DD2F7AA/5DDC92C2" Ref="D?"  Part="1"
-AR Path="/5DDC92C2" Ref="D2"  Part="1"
-F 0 "D2" H 14691 7516 50  0000 C CNN
-F 1 "LED" H 14691 7425 50  0000 C CNN
-F 2 "pecanpico:LED_0402" H 14700 7300 50  0001 C CNN
-F 3 "~" H 14700 7300 50  0001 C CNN
-	1    14700 7300
-	1    0    0    -1
-$EndComp
-Wire Wire Line
-	14550 7300 14350 7300
-Wire Wire Line
-	14850 7300 14950 7300
-Wire Wire Line
-	14950 7300 14950 7200
-$Comp
-L pecanpico:+GPS #PWR?
-U 1 1 5DDC92CB
-P 14950 7200
-AR Path="/5DD2F7AA/5DDC92CB" Ref="#PWR?"  Part="1"
-AR Path="/5DDC92CB" Ref="#PWR0154"  Part="1"
-F 0 "#PWR0154" H 14950 7050 50  0001 C CNN
-F 1 "+GPS" V 14950 7325 50  0000 L CNN
-F 2 "" H 14950 7200 50  0000 C CNN
-F 3 "" H 14950 7200 50  0000 C CNN
-	1    14950 7200
-	1    0    0    -1
-$EndComp
-Text Label 14750 6600 2    50   ~ 0
-SCK2
 $Comp
 L pecanpico:SIP3243x IC?
@@
 Wire Wire Line
 	8600 9900 8500 9900
-Wire Wire Line
-	8500 9900 8500 9800
-$Comp
-L pecanpico:+1V8 #PWR?
-U 1 1 5DDE750E
-P 8500 9800
-AR Path="/5DD2F7AA/5DDE750E" Ref="#PWR?"  Part="1"
-AR Path="/5DDE750E" Ref="#PWR0157"  Part="1"
-F 0 "#PWR0157" H 8500 9650 50  0001 C CNN
-F 1 "+1V8" H 8500 9950 50  0000 C CNN
-F 2 "" H 8500 9800 50  0001 C CNN
-F 3 "" H 8500 9800 50  0001 C CNN
-	1    8500 9800
-	1    0    0    -1
-$EndComp
 Wire Wire Line
 	8600 10200 8300 10200
@@
 	1    0    0    -1
 $EndComp
+$Comp
+L power:+3.3V #PWR?
+U 1 1 5DED6E47
+P 8500 9800
+AR Path="/5D5B165E/5DED6E47" Ref="#PWR?"  Part="1"
+AR Path="/5D5B15F7/5DED6E47" Ref="#PWR?"  Part="1"
+AR Path="/5DED6E47" Ref="#PWR0110"  Part="1"
+F 0 "#PWR0110" H 8500 9650 50  0001 C CNN
+F 1 "+3.3V" H 8515 9973 50  0000 C CNN
+F 2 "" H 8500 9800 50  0001 C CNN
+F 3 "" H 8500 9800 50  0001 C CNN
+	1    8500 9800
+	1    0    0    -1
+$EndComp
+Wire Wire Line
+	8500 9800 8500 9900
+NoConn ~ 14350 5800
+NoConn ~ 14350 5900
+NoConn ~ 14350 6000
+NoConn ~ 14350 6100
+NoConn ~ 14350 6200
+NoConn ~ 14350 6300
+NoConn ~ 12950 7050
+NoConn ~ 12950 7300
+NoConn ~ 12950 7400
+Wire Wire Line
+	14350 6600 15150 6600
+Wire Wire Line
+	14350 6500 15150 6500
+Text Label 15150 6600 2    50   ~ 0
+I2C1_SCL
+Text Label 15150 6500 2    50   ~ 0
+I2C1_SDA
+NoConn ~ 14350 6800
+Wire Wire Line
+	14350 7000 15150 7000
+Text Label 15150 7000 2    50   ~ 0
+GPS_SAFEBOOT
+NoConn ~ 14350 6700
+NoConn ~ 14350 7100
+NoConn ~ 14350 7400
+Wire Wire Line
+	7150 3300 7800 3300
+Text Label 7800 3300 2    50   ~ 0
+GPS_EN
+NoConn ~ 7150 3100
+NoConn ~ 7150 3200
+$Comp
+L power:PWR_FLAG #FLG0101
+U 1 1 5E0E0060
+P 1300 7950
+F 0 "#FLG0101" H 1300 8025 50  0001 C CNN
+F 1 "PWR_FLAG" H 1300 8123 50  0000 C CNN
+F 2 "" H 1300 7950 50  0001 C CNN
+F 3 "~" H 1300 7950 50  0001 C CNN
+	1    1300 7950
+	1    0    0    -1
+$EndComp
+Connection ~ 1300 7950
+Wire Wire Line
+	1300 7950 2400 7950
+Wire Wire Line
+	2400 7950 2400 7450
+Wire Wire Line
+	1250 8350 1800 8350
+Wire Wire Line
+	1800 8750 1800 8350
+$Comp
+L power:GND #PWR0102
+U 1 1 5DEE121A
+P 1800 8750
+F 0 "#PWR0102" H 1800 8500 50  0001 C CNN
+F 1 "GND" H 1805 8577 50  0000 C CNN
+F 2 "" H 1800 8750 50  0001 C CNN
+F 3 "" H 1800 8750 50  0001 C CNN
+	1    1800 8750
+	1    0    0    -1
+$EndComp
+Wire Wire Line
+	2400 7950 2400 8050
+Connection ~ 2400 7950
+$Comp
+L power:GND #PWR0119
+U 1 1 5E15E5A3
+P 2400 8750
+F 0 "#PWR0119" H 2400 8500 50  0001 C CNN
+F 1 "GND" H 2405 8577 50  0000 C CNN
+F 2 "" H 2400 8750 50  0001 C CNN
+F 3 "" H 2400 8750 50  0001 C CNN
+	1    2400 8750
+	1    0    0    -1
+$EndComp
+$Comp
+L Device:R R?
+U 1 1 5E16906A
+P 2400 8200
+AR Path="/5D5B15F7/5E16906A" Ref="R?"  Part="1"
+AR Path="/5E16906A" Ref="R2"  Part="1"
+F 0 "R2" H 2470 8246 50  0000 L CNN
+F 1 "10K" H 2470 8155 50  0000 L CNN
+F 2 "Resistor_SMD:R_0402_1005Metric" V 2330 8200 50  0001 C CNN
+F 3 "~" H 2400 8200 50  0001 C CNN
+	1    2400 8200
+	1    0    0    -1
+$EndComp
+Wire Wire Line
+	2400 8350 2400 8400
+$Comp
+L Device:R R?
+U 1 1 5E1696E7
+P 2400 8600
+AR Path="/5D5B15F7/5E1696E7" Ref="R?"  Part="1"
+AR Path="/5E1696E7" Ref="R9"  Part="1"
+F 0 "R9" H 2470 8646 50  0000 L CNN
+F 1 "10K" H 2470 8555 50  0000 L CNN
+F 2 "Resistor_SMD:R_0402_1005Metric" V 2330 8600 50  0001 C CNN
+F 3 "~" H 2400 8600 50  0001 C CNN
+	1    2400 8600
+	1    0    0    -1
+$EndComp
+Connection ~ 2400 8400
+Wire Wire Line
+	2400 8400 2400 8450
+Text Label 3400 8400 2    50   ~ 0
+V_SOLAR
+Wire Wire Line
+	2400 8400 3400 8400
+Wire Notes Line
+	11100 650  11100 11200
+Wire Notes Line
+	500  11200 11100 11200
+Text Notes 7300 11000 0    50   ~ 0
+Switch to turn on and off GPS\n
+Text Notes 7250 9000 0    50   ~ 0
+MPPT + boost converter to charge battery
+NoConn ~ 7150 3800
+NoConn ~ 14350 7300
+Text Label 12300 7200 0    50   ~ 0
+GPS_EXTINT
+Wire Wire Line
+	12950 7200 12300 7200
+NoConn ~ 8100 8250
+NoConn ~ 8050 8100
+$Comp
+L Device:Battery_Cell BT?
+U 1 1 5E286112
+P 10350 8050
+F 0 "BT?" H 10468 8146 50  0000 L CNN
+F 1 "Battery_Cell" H 10468 8055 50  0000 L CNN
+F 2 "" V 10350 8110 50  0001 C CNN
+F 3 "~" V 10350 8110 50  0001 C CNN
+	1    10350 8050
+	1    0    0    -1
+$EndComp
+$Comp
+L pecanpico:GND #PWR?
+U 1 1 5E287D9D
+P 10350 8450
+AR Path="/5DD2F7AA/5E287D9D" Ref="#PWR?"  Part="1"
+AR Path="/5E287D9D" Ref="#PWR?"  Part="1"
+F 0 "#PWR?" H 10350 8200 50  0001 C CNN
+F 1 "GND" H 10350 8300 50  0000 C CNN
+F 2 "" H 10350 8450 50  0001 C CNN
+F 3 "" H 10350 8450 50  0001 C CNN
+	1    10350 8450
+	1    0    0    -1
+$EndComp
+Wire Wire Line
+	10350 8450 10350 8150
+Wire Wire Line
+	10000 7550 10350 7550
+Wire Wire Line
+	10350 7550 10350 7850
 $EndSCHEMATC

Commit message: changed the layout of schematic of "b" variant to save space
Other:
- moved on the sheet: C14, R4, R5, U6

Commit message: updated circuit of b variant for low power voltage measurment. Made a variant tcxo enable controllable
Parts:
- removed BT?: Battery_Cell, symbol Device:Battery_Cell
- removed C16: 1n, Capacitor_SMD:C_0402_1005Metric, symbol pecanpico:C
- removed C17, C3: 22u, Capacitor_SMD:C_0805_2012Metric, symbol pecanpico:C
- removed C18: 100n, Capacitor_SMD:C_0402_1005Metric, symbol pecanpico:C
- removed IC8: SIP32431DNP3-T1GE4, pecanpico:DFN-4-1EP_1.2x1.6mm_P0.5mm_EP, symbol pecanpico:SIP3243x
- removed IC9: ZOE-M8G/B, pecanpico:ZOE-M8, symbol pecanpico:ZOE-M8G
- removed L7: XFL2006-472MEB, pecanpico:XFL20xx, symbol pecanpico:L_Small
- removed R1, R8: R, Resistor_SMD:R_0402_1005Metric, symbol pecanpico:R
- added AE3: GPS Antenna, Connector_Wire:SolderWirePad_1x01_Drill0.8mm, symbol flight-computer:GPS_Antenna
- added C12, C2, C8: 10uF, Capacitor_SMD:C_0603_1608Metric, symbol Device:C_Small
- added C13, C18, C6: 100nF, Capacitor_SMD:C_0402_1005Metric, symbol Device:C_Small
- added C15: 1uF, Capacitor_SMD:C_0603_1608Metric, symbol Device:C_Small
- added C16, C4: 1nF, Capacitor_SMD:C_0402_1005Metric, symbol Device:C_Small
- added C17: 22uF, Capacitor_SMD:C_0805_2012Metric, symbol Device:C_Small
- added C3: 4.7uF, Capacitor_SMD:C_0805_2012Metric, symbol Device:C_Small
- added D2: D_Schottky, Diode_SMD:D_0402_1005Metric, symbol Device:D_Schottky
- added J5: BATT_GND, Connector_Wire:SolderWirePad_1x01_Drill0.8mm, symbol Connector_Generic:Conn_01x01
- added L2: 2.2uH, Inductor_SMD:L_Taiyo-Yuden_NR-30xx, symbol Device:L
- added L3: 10uH, Inductor_coilcraft:LPS3015, symbol Device:L
- added Q1, Q2: Q_PMOS_DGS, Package_TO_SOT_SMD:SOT-23, symbol Device:Q_PMOS_DGS
- added R1, R17: 10K, Resistor_SMD:R_0402_1005Metric, symbol Device:R
- added R10, R11, R8: 1K, Resistor_SMD:R_0402_1005Metric, symbol Device:R
- added R12: 1Ohm, Resistor_SMD:R_0402_1005Metric, symbol Device:R
- added R13: 10M, Resistor_SMD:R_0402_1005Metric, symbol Device:R
- added R14: 5.1M, Resistor_SMD:R_0402_1005Metric, symbol Device:R
- added R15, R16: 100K, Resistor_SMD:R_0402_1005Metric, symbol Device:R
- added U2: TPS62740, Package_SON:WSON-12-1EP_3x2mm_P0.5mm_EP1x2.65, symbol flight-computer:TPS62740
- added U4: MAX-M8C, RF_GPS:ublox_MAX, symbol RF_GPS:MAX-M8C
- C10: Cost (none) -> 0.07
- J1: footprint femto_footprints:special_test_pads -> flight-computer:special_test_pads
- J4: value Conn_01x01 -> BATT_V+; footprint Connector_PinHeader_1.27mm:PinHeader_1x01_P1.27mm_Vertical -> Connector_Wire:SolderWirePad_1x01_Drill0.8mm
- R2, R9: value 10K -> 100K
Connections:
- net +SOL: now also C3.1, L3.2, Q2.3 (S), R17.1, R8.1; no longer IC7.3 (LX), R2.1
- net GND: now also IC7.2 (GND), C12.2, C16.2, C17.1, C2.2, C3.2, C4.2, C6.2, C8.2, D2.2 (A), J5.1 (Pin_1), R14.1, R16.2, U2.3 (GND), U2.8 (VSEL4), U2.9 (VSEL3), U4.1 (GND), U4.10 (GND), U4.12 (GND), U4.13 (LNA_EN); no longer IC7.1 (MPP-SET)
- net GPS_EXTINT: now also U4.5 (EXTINT)
- net GPS_SAFEBOOT: now also U4.18 (~SAFEBOOT)
- net I2C1_SCL: now also U4.17 (SCL)
- net I2C1_SDA: now also U4.16 (SDA)
- net GPS_TIMEPULSE: now reaches U3.15 (PB14/SPI2_MISO)
- net GPS_TIMEPULSE: now also U4.4 (TIMEPULSE)
- net SOL_PWR_MEASURE: now reaches U3.18 (PA10/USART1_RX)
- net SOL_PWR_MEASURE: now also C18.2
- net BATT_PWR_MEASURE: now reaches U3.19 (PA9/USART1_TX)
- net BATT_PWR_MEASURE: now also C13.2
- net BATT_VOLTS: now reaches U3.23 (PA3/ADC3)
- net BATT_VOLTS: now also R15.2, R16.1
- net TCXO_EN: now reaches U3.40 (PB5/LPTIM1_IN1)
- net TCXO_EN: now also U3.48 (VDD_TCXO)
- net at IC7.5 (VCTRL): now also C16.1, R13.1, R14.2
- net at IC7.6 (ICTRL-): now also C15.2, R11.2
- net at IC7.7 (ICTRL+): now also C15.1, R10.2
- net +BATT: now reaches J4.1 (Pin_1)
- net +BATT: now also C2.1, D2.1 (K), Q1.3 (S), R1.1, R11.1, R12.2, R13.2, U2.1 (VIN), U2.10 (VSEL2), U2.11 (VSEL1), U2.12 (EN)
- net +3V3 renamed VCC
- net VCC: now also C12.1, C6.1, C8.1, L2.1, U2.5 (VOUT), U4.6 (V_BCKP), U4.7 (VCC_IO), U4.8 (VCC), U4.9 (~RESET); no longer C14.1, IC7.4 (VOUT), R4.1, R5.1, U3.48 (VDD_TCXO), U6.1 (VDD), U6.2 (PS)
- net GPS_EN renamed SENSOR_EN
- net SENSOR_EN: now also U2.4 (CTRL)
- net V_SOLAR renamed SOLAR_VOLTS
- new net: AE3.1 (A), U4.11 (RF_IN)
- new net: C4.1, IC7.1 (MPP-SET), R8.2
- new net: C18.1, Q2.2 (G), R17.2
- new net: L2.2, U2.2 (SW)
- new net: Q2.1 (D), R2.1
- new net: C17.2, IC7.4 (VOUT), R10.1, R12.1
- new net: IC7.3 (LX), L3.1
- new net: Q1.1 (D), R15.1
- new net: C13.1, Q1.2 (G), R1.2
- new net SENSOR_VCC: C14.1, R4.1, R5.1, U2.6 (LOAD), U6.1 (VDD), U6.2 (PS)
- no-connect marks 46 -> 30
Other:
- note added: "Buck coverter to bring battery voltage down to voltage for GPS and ABZ module"
- note added: "I2C pullup resistors"
- note added: "Must adjust values of VSEL pin connections to target output voltage."
- note added: "Ultra Low current Solar and Battery voltage measurment"
- note removed: "Switch to turn on and off GPS\n"
- moved on the sheet: AE1, C1, C10, C5, C7, IC7, J2, R2, R4, R9, U3
