File: prototype/hardware/Kicad/Picotracker V1.1b/circuit board design.kicad_pcb (KiCad board)
At the start: 2 copper layers, 47.4 x 20.1 mm, 55 parts, among them IC7 SPV1040, J1 Conn_01x10, J6 ICSS LOGO, Q1 Q_PMOS_GSD, SW1 SW_Push, U2 TPS62740, U3 CMWX1ZZABZ-078, U4 MAX-M8C, U6 MS5607-02BA

Commit message: finished lora tracker v1.1 for a and b variants
Parts:
- renumbered GND to J2, +SOL to J3, +BATT to J4, GND to J5
Other:
- board text added: "+BATT"
- board text added: "+SOL"
