File: Current Tracker Prototype/hardware/Kicad/Picotracker V1.2b/circuit board design.sch (KiCad schematic (older format))
At the start: 54 parts, among them IC7 SPV1040, J1 Conn_01x10, J2 GND, J3 +SOL, J4 BATT_V+, J5 BATT_GND, J6 ICSS LOGO, J7 Conn_01x01, J8 Conn_01x01, Q1 Q_PMOS_GSD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

Commit message: connected pin 1 to pin 8 on SPV1040
Connections:
- wire segments 214 -> 217
- no-connect marks 35 -> 34
Changed lines of the file:
@@
 Wire Wire Line
 	1550 6050 1550 6500
-NoConn ~ 12600 2000
 $Comp
 L Device:C_Small C?
@@
 	12200 1850 12300 1850
 Wire Wire Line
-	12200 2350 12600 2350
+	12200 2350 12400 2350
 $Comp
 L Device:C_Small C?
@@
 AR Path="/5DC7C9E7" Ref="#PWR09"  Part="1"
 F 0 "#PWR09" H 12500 1950 50  0001 C CNN
-F 1 "GND" H 12400 2100 50  0000 C CNN
+F 1 "GND" H 12500 2250 50  0000 C CNN
 F 2 "" H 12500 2200 50  0001 C CNN
 F 3 "" H 12500 2200 50  0001 C CNN
@@
 Wire Wire Line
 	6700 5250 8150 5250
+Wire Wire Line
+	12600 2000 12400 2000
+Wire Wire Line
+	12400 2000 12400 2350
+Connection ~ 12400 2350
+Wire Wire Line
+	12400 2350 12600 2350
 $EndSCHEMATC

Commit message: Update circuit board design.sch
Connections:
- net labels added: GPS_EXTINT
- wire segments 217 -> 219
- no-connect marks 34 -> 32
Changed lines of the file:
@@
 Wire Wire Line
 	13000 7750 11800 7750
-NoConn ~ 13000 7550
 Text Label 7350 3850 2    50   ~ 0
 GPS_TIMEPULSE
 Wire Wire Line
 	6700 3850 7350 3850
-NoConn ~ 6700 3750
 NoConn ~ 6700 3150
 Wire Wire Line
@@
 USART1_TX
 NoConn ~ 13600 6650
-$Comp
-L Device:Q_PMOS_GSD Q1
-U 1 1 5DF9440B
-P 7950 7800
-F 0 "Q1" H 8156 7846 50  0000 L CNN
-F 1 "Q_PMOS_GSD" H 8156 7755 50  0000 L CNN
-F 2 "Package_TO_SOT_SMD:SOT-23" H 8150 7900 50  0001 C CNN
-F 3 "~" H 7950 7800 50  0001 C CNN
-	1    7950 7800
-	1    0    0    -1
-$EndComp
 Wire Wire Line
 	5900 2450 5900 2150
@@
 Wire Wire Line
 	12400 2350 12600 2350
+$Comp
+L Device:Q_PMOS_GSD Q1
+U 1 1 5DF9440B
+P 7950 7800
+F 0 "Q1" H 8156 7846 50  0000 L CNN
+F 1 "Q_PMOS_GSD" H 8156 7755 50  0000 L CNN
+F 2 "Package_TO_SOT_SMD:SOT-23" H 8150 7900 50  0001 C CNN
+F 3 "~" H 7950 7800 50  0001 C CNN
+	1    7950 7800
+	1    0    0    1
+$EndComp
+Text Label 7350 3750 2    50   ~ 0
+GPS_EXTINT
+Wire Wire Line
+	7350 3750 6700 3750
+Wire Wire Line
+	12300 7550 13000 7550
+Text Label 12300 7550 0    50   ~ 0
+GPS_EXTINT
 $EndSCHEMATC
