File: Current Tracker Prototype/hardware/Kicad/Picotracker V1.2b/_autosave-circuit board design.kicad_pcb (KiCad board)
At the start: 2 copper layers, 47.4 x 20.1 mm, 53 parts, among them IC7 SPV1040, J1 Conn_01x10, J2 GND, J3 +SOL, J4 Batt connection, J6 ICSS LOGO, J7 Conn_01x01, J8 Conn_01x01, Q1 Q_PMOS_GSD, SW1 SW_Push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

Commit message: finished designs of v1.2 a and b
Routing:
- net GND: vias 45 -> 44
Changed lines of the file:
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@@
     (thickness 0.6)
     (drawings 28)
-    (tracks 555)
+    (tracks 554)
     (zones 0)
     (modules 53)
@@
       (drillshape 0)
       (scaleselection 1)
-      (outputdirectory "D:/Long term storage and temp/dead weight program downloads/lora tracker outputs/loratracker v1.1b/"))
+      (outputdirectory "D:/Long term storage and temp/dead weight program downloads/lora tracker outputs/loratracker v1.2b/"))
   )
   (net 0 "")
@@
   (via (at 267.589 170.434) (size 0.8) (drill 0.4) (layers F.Cu B.Cu) (net 1))
   (via (at 268.859 170.942) (size 0.8) (drill 0.4) (layers F.Cu B.Cu) (net 1))
-  (via (at 267.208 171.45) (size 0.8) (drill 0.4) (layers F.Cu B.Cu) (net 1))
   (segment (start 300.619 162.193) (end 300.619 161.993) (width 0.25) (layer F.Cu) (net 2) (status 30))
   (via (at 303.784 168.529) (size 0.8) (drill 0.4) (layers F.Cu B.Cu) (net 2))
@@
   (segment (start 290.432484 177.364509) (end 288.947212 175.879237) (width 0.25) (layer F.Cu) (net 11))
   (segment (start 293.004503 177.364509) (end 290.432484 177.364509) (width 0.25) (layer F.Cu) (net 11))
-  (segment (start 295.529 178.689) (end 294.328994 178.689) (width 0.25) (layer F.Cu) (net 11))
+  (segment (start 295.529 178.689) (end 294.328994 178.689) (width 0.25) (layer F.Cu) (net 11) (status 10))
   (segment (start 294.328994 178.689) (end 293.004503 177.364509) (width 0.25) (layer F.Cu) (net 11))
   (segment (start 293.093 175.675) (end 293.093 176.53) (width 0.25) (layer F.Cu) (net 12) (status 20))
