File: Current Tracker Prototype/hardware/Kicad/Picotracker V1.2b/_autosave-circuit board design.sch (KiCad schematic (older format))
At the start: 53 parts, among them IC7 SPV1040, J1 Conn_01x10, J2 GND, J3 +SOL, J4 Batt connection, J6 ICSS LOGO, J7 Conn_01x01, J8 Conn_01x01, Q1 Q_PMOS_GSD, SW1 SW_Push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

Commit message: finished designs of v1.2 a and b
Parts:
- J4: footprint Connector_Wire:SolderWirePad_1x01_Drill0.8mm -> Connector_PinHeader_2.54mm:PinHeader_1x02_P2.54mm_Vertical
Changed lines of the file:
@@
 F 0 "J4" H 9880 10142 50  0000 L CNN
 F 1 "Batt connection" H 9880 10051 50  0000 L CNN
-F 2 "Connector_Wire:SolderWirePad_1x01_Drill0.8mm" H 9800 10100 50  0001 C CNN
+F 2 "Connector_PinHeader_2.54mm:PinHeader_1x02_P2.54mm_Vertical" H 9800 10100 50  0001 C CNN
 F 3 "~" H 9800 10100 50  0001 C CNN
 	1    9800 10100
