File: Current Tracker Prototype/hardware/Kicad/Picotracker V1.3a/circuit board design.sch (KiCad schematic (older format))
At the start: 30 parts, among them J1 Conn_01x10, J2 GND, J3 3.3V, J4 ICSS Logo, J5 Conn_01x01, Q1 IRLML6402, SW1 SW_Push, U1 MAX-M8C, U3 CMWX1ZZABZ-078, U6 MS5607-02BA

Commit message: Makeing board 1.3a (#30)
* pull gps ddc and uart pins out to side test points
* connect stm32 reset line to vcc via resistor
* connect stm32 to gps via usart2
* put in the test points
* put in test point to switched gps power supply
* update annotation
* put test point name labels
* put in solder jumper for uart. Connected i2c as well
* changed the lora antenna pad to rectangular
* made seperate custom abz foot print
* made seperate folder for 1.3a design
* put in pdf schematic of 1.3a

Co-authored-by: MedadRufus <mailto@medadnewman.co.uk>
Parts:
- removed C1: 100nF, Capacitor_SMD:C_0402_1005Metric, symbol Device:C_Small
- removed R7: 100K, Resistor_SMD:R_0402_1005Metric, symbol Device:R
- removed SW1: SW_Push, flight-computer:EVPAWCD4A, symbol Switch:SW_Push
- added JP1, JP2: SolderJumper_2_Open, Jumper:SolderJumper-2_P1.3mm_Open_RoundedPad1.0x1.5mm, symbol Jumper:SolderJumper_2_Open
- added R9: 10K, Resistor_SMD:R_0402_1005Metric, symbol circuit-board-design-rescue:R-Device
- added TP1, TP2, TP3, TP4, TP5, TP6, TP7, TP8, TP9: TestPoint, TestPoint:TestPoint_Pad_D1.0mm, symbol Connector:TestPoint
- AE1: footprint Connector_Wire:SolderWirePad_1x01_Drill0.8mm -> pico_tracker:SolderWirePad_1x01_Drill0.8mm_square; symbol Device:Antenna -> circuit-board-design-rescue:Antenna-Device
- C10, C12, C13, C14, C5, C7: symbol Device:C_Small -> circuit-board-design-rescue:C_Small-Device
- D1: symbol Device:LED -> circuit-board-design-rescue:LED-Device
- J1: symbol Connector_Generic:Conn_01x10 -> circuit-board-design-rescue:Conn_01x10-Connector_Generic
- J2, J3, J4, J5, SolarCellMount1, StringHole1: symbol Connector_Generic:Conn_01x01 -> circuit-board-design-rescue:Conn_01x01-Connector_Generic
- Q1: symbol Transistor_FET:IRLML6402 -> circuit-board-design-rescue:IRLML6402-Transistor_FET
- R1, R2, R3, R4, R5, R6, R8: symbol Device:R -> circuit-board-design-rescue:R-Device
- U1: symbol RF_GPS:MAX-M8C -> circuit-board-design-rescue:MAX-M8C-RF_GPS
- U3: footprint RF_Module:CMWX1ZZABZ -> pico_tracker:CMWX1ZZABZ_custom; symbol RF_Module:CMWX1ZZABZ-078 -> circuit-board-design-rescue:CMWX1ZZABZ-078-RF_Module
- U6: symbol Sensor_Pressure:MS5607-02BA -> circuit-board-design-rescue:MS5607-02BA-Sensor_Pressure
Connections:
- net labels added: USART2_RX, USART2_TX
- net labels removed: SWITCH
- wire segments 134 -> 147
- no-connect marks 31 -> 25
Other:
- note removed: "User interface button\n"
