File: hardware/Kicad/Picotracker V1.3a/circuit board design.sch (KiCad schematic (older format))
At the start: 39 parts, among them J1 Conn_01x10, J2 GND, J3 3.3V, J4 ICSS Logo, J5 Conn_01x01, Q1 IRLML6402, U1 MAX-M8C, U3 CMWX1ZZABZ-078, U6 MS5607-02BA

Commit message: Change GPS antenna pad to the same as the lora pad
Use a rectangular pad for GPS antenna. Much stronger connection.
Put in test pad on GPS timepulse.
Parts:
- removed AE1: Lora Antenna, pico_tracker:SolderWirePad_1x01_Drill0.8mm_square, symbol circuit-board-design-rescue:Antenna-Device
- added AE1: GPS Antenna, pico_tracker:custom_antenna_pad, symbol flight-computer:GPS_Antenna
- added TP?: TestPoint, TestPoint:TestPoint_Pad_D1.0mm, symbol Connector:TestPoint
- AE2: footprint Connector_Wire:SolderWirePad_1x01_Drill0.8mm -> pico_tracker:custom_antenna_pad
Connections:
- wire segments 147 -> 149
Changed lines of the file:
@@
 EESchema Schematic File Version 4
-LIBS:circuit board design-cache
 EELAYER 29 0
 EELAYER END
@@
 	14050 8200 14050 8350
 Wire Wire Line
-	14650 7800 15500 7800
-Text Label 15500 7800 2    50   ~ 0
-GPS_TIMEPULSE
+	14650 7800 15100 7800
 Wire Wire Line
 	7150 3800 7800 3800
@@
 $EndComp
 $Comp
-L circuit-board-design-rescue:Antenna-Device AE1
-U 1 1 5DE442FF
-P 8600 4850
-F 0 "AE1" H 8680 4839 50  0000 L CNN
-F 1 "Lora Antenna" H 8680 4748 50  0000 L CNN
-F 2 "pico_tracker:SolderWirePad_1x01_Drill0.8mm_square" H 8600 4850 50  0001 C CNN
-F 3 "~" H 8600 4850 50  0001 C CNN
-	1    8600 4850
-	1    0    0    -1
-$EndComp
-$Comp
 L flight-computer:GPS_Antenna AE2
 U 1 1 5DDA946B
@@
 F 0 "AE2" H 15380 7139 50  0000 L CNN
 F 1 "GPS Antenna" H 15380 7048 50  0000 L CNN
-F 2 "Connector_Wire:SolderWirePad_1x01_Drill0.8mm" H 15300 7150 50  0001 C CNN
+F 2 "pico_tracker:custom_antenna_pad" H 15300 7150 50  0001 C CNN
 F 3 "~" H 15300 7150 50  0001 C CNN
 	1    15300 7150
@@
 Wire Wire Line
 	8600 5350 8600 5950
+$Comp
+L flight-computer:GPS_Antenna AE1
+U 1 1 6018FBE3
+P 8600 4850
+F 0 "AE1" H 8680 4839 50  0000 L CNN
+F 1 "GPS Antenna" H 8680 4748 50  0000 L CNN
+F 2 "pico_tracker:custom_antenna_pad" H 8600 4850 50  0001 C CNN
+F 3 "~" H 8600 4850 50  0001 C CNN
+	1    8600 4850
+	1    0    0    -1
+$EndComp
+$Comp
+L Connector:TestPoint TP?
+U 1 1 6019818B
+P 15100 8050
+F 0 "TP?" H 15158 8168 50  0000 L CNN
+F 1 "TestPoint" H 15150 8100 50  0000 L CNN
+F 2 "TestPoint:TestPoint_Pad_D1.0mm" H 15300 8050 50  0001 C CNN
+F 3 "~" H 15300 8050 50  0001 C CNN
+	1    15100 8050
+	-1   0    0    1
+$EndComp
+Wire Wire Line
+	15100 8050 15100 7800
+Text Label 15750 7800 2    50   ~ 0
+GPS_TIMEPULSE
+Wire Wire Line
+	15100 7800 15750 7800
+Connection ~ 15100 7800
 $EndSCHEMATC

Commit message: put in test point on GPS pps pin
Parts:
- gave numbers to parts that had none: 1
Changed lines of the file:
@@
 $EndComp
 $Comp
-L Connector:TestPoint TP?
+L Connector:TestPoint TP10
 U 1 1 6019818B
 P 15100 8050
-F 0 "TP?" H 15158 8168 50  0000 L CNN
+F 0 "TP10" H 15158 8168 50  0000 L CNN
 F 1 "TestPoint" H 15150 8100 50  0000 L CNN
 F 2 "TestPoint:TestPoint_Pad_D1.0mm" H 15300 8050 50  0001 C CNN
